Commit message: new update map gazebo

File: description/robot_core.xacro (robot description, xacro)
@@ -4,4 +4,7 @@
     <material name="white">
         <color rgba="1 1 1 1"/>
+    </material>
+    <material name="red">
+        <color rgba="0 1 0 1"/>
     </material>
     <material name="orange">
